File: oae/adc_communications.kicad_sch (KiCad schematic)
At the start: 3 parts

Commit message: Add resistors to power supply
Parts:
- R1: footprint (none) -> Resistor_SMD:R_0603_1608Metric_Pad0.98x0.95mm_HandSolder
Changed lines of the file:
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@@
       (effects (font (size 1.27 1.27)) (justify left))
     )
-    (property "Footprint" "" (at 95.25 76.2 0)
+    (property "Footprint" "Resistor_SMD:R_0603_1608Metric_Pad0.98x0.95mm_HandSolder" (at 95.25 76.2 0)
       (effects (font (size 1.27 1.27)) hide)
     )
